Commit message: enable arm ctrl with joypad and adjust transformation between 3d camera and arm

File: raw_robots/raw_hardware_config/youbot/urdf/youbot.urdf.xacro (robot description, xacro)
@@ -64,5 +64,5 @@
   <!-- 3D camera on tower -->
   <xacro:kinect_camera name="openni" parent="tower_link">
-    <origin xyz="0.0509 -0.03 0.49" rpy="0 0.545 0" />
+    <origin xyz="0.0109 -0.03 0.49" rpy="0 0.545 0.08" />
   </xacro:kinect_camera>
   <!-- Microsoft LifeCam on gripper -->
